Commit message: In this version the robot arm can be moved! This is the first working version. This should now be taken and put onto the MiR200. Add fixed joint to world link. Add common.xacro to ur robot so gazebo plugin is spawned Add controller_list file. controller list and spawned arm controller must be in different file! Added joint_names.yaml. Not sure if needed, should be in ros_controllers.yaml Fixed bug where planner "NONE" was not found Removed controller_list from ros_controllers file. Has nothing to do there. must be in different yaml. Added arm_controller in ros_controllers. Fixed bug in sensors_3d file Changed the srdf moveit file from joints to links like in the universal robot repo example Added remapping because arm_controller has a name. Could try without name so no remapping is needed Removed obsolete stuff like the db logging Fixed wrong parameter at rviz launch Changed loading xacro from textfile to xacro param Added rviz config. Could be done different, but this works Added the controllers  in ros_controllers.launch that should be spawned to control the robot Added the controllers.yaml with controller_list to the controller_manager.launch

File: mir_ur5_description/urdf/ur5_robot.urdf.xacro (robot description, xacro)
@@ -5,8 +5,14 @@
   <xacro:arg name="transmission_hw_interface" default="hardware_interface/PositionJointInterface"/>
   <!-- common stuff -->
-  <!-- <xacro:include filename="$(find ur_description)/urdf/common.gazebo.xacro" /> -->
+  <xacro:include filename="$(find ur_description)/urdf/common.gazebo.xacro" />
   <!-- include of the xacro file -->
   <xacro:include filename="$(find mir_ur5_description)/urdf/ur5.urdf.xacro" />
   <!-- arm -->
   <xacro:ur5_robot prefix="" joint_limited="false" transmission_hw_interface="$(arg transmission_hw_interface)"/>
+  <link name="world" />
+  <joint name="world_joint" type="fixed">
+    <parent link="world" />
+    <child link = "base_link_ur5" />
+    <origin xyz="0.0 0.0 0.0" rpy="0.0 0.0 0.0" />
+  </joint>
 </robot>

Commit message: Need to get the whole urdf file for configuration of moveit package, otherwise the semantic file that is loaded throws errors that it is not same as currently loaded urdf file (when configured with only ur5 urdf)

File: mir_ur5_description/urdf/ur5_robot.urdf.xacro (robot description, xacro)
@@ -5,14 +5,14 @@
   <xacro:arg name="transmission_hw_interface" default="hardware_interface/PositionJointInterface"/>
   <!-- common stuff -->
-  <xacro:include filename="$(find ur_description)/urdf/common.gazebo.xacro" />
+  <!-- <xacro:include filename="$(find ur_description)/urdf/common.gazebo.xacro" /> -->
   <!-- include of the xacro file -->
   <xacro:include filename="$(find mir_ur5_description)/urdf/ur5.urdf.xacro" />
   <!-- arm -->
   <xacro:ur5_robot prefix="" joint_limited="false" transmission_hw_interface="$(arg transmission_hw_interface)"/>
-  <link name="world" />
+  <!-- <link name="world" />
   <joint name="world_joint" type="fixed">
     <parent link="world" />
     <child link = "base_link_ur5" />
     <origin xyz="0.0 0.0 0.0" rpy="0.0 0.0 0.0" />
-  </joint>
+  </joint> -->
 </robot>
