Commit message: Added new stl file for the MiR200 base new stl also contains base where robot is bolted on Changed MiR xacro so the new stl is scaled correctly Changed mesh to new file Changed rotation because looks like the axis are different to the last stl file that was loaded

File: mir_ur5_description/urdf/mir_200_v1.urdf.xacro (robot description, xacro)
@@ -137,14 +137,14 @@
       </xacro:box_inertial>
       <visual>
-        <origin xyz="${mir_200_act_wheel_dx} 0 0" rpy="0 0 0" />
-        <geometry>
-          <mesh filename="package://mir_description/meshes/visual/MIR200_base.stl" />
+        <origin xyz="${mir_200_act_wheel_dx} 0 0" rpy="${pi/2} 0 ${pi/2}" />
+        <geometry>
+          <mesh filename="package://mir_ur5_description/meshes/MiR200_UR5_base.stl" scale="0.001 0.001 0.001"/> <!--Scale is necessary because stl was generated in mm (correct dimensions) but stl has no measurements and mm are interpreted as m in gazebo-->
         </geometry>
         <xacro:insert_block name="material_white" />
       </visual>
       <collision>
-        <origin xyz="${mir_200_act_wheel_dx} 0 0" rpy="0 0 0" />
-        <geometry>
-          <mesh filename="package://mir_description/meshes/collision/MIR200_base.stl" />
+        <origin xyz="${mir_200_act_wheel_dx} 0 0" rpy="${pi/2} 0 ${pi/2}" />
+        <geometry>
+          <mesh filename="package://mir_ur5_description/meshes/MiR200_UR5_base.stl" scale="0.001 0.001 0.001"/> <!--Scale is necessary because stl was generated in mm (correct dimensions) but stl has no measurements and mm are interpreted as m in gazebo-->
         </geometry>
       </collision>

Commit message: Changed names of links in the ur5 robot

File: mir_ur5_description/urdf/mir_200_v1.urdf.xacro (robot description, xacro)
@@ -154,6 +154,6 @@
     </gazebo>
     <!--Include the UR5 into the model. The position of the model was measured usind laser scanner. See Florians master thesis-->
-    <xacro:include filename="$(find ur_description)/urdf/ur5.urdf.xacro"/>
-    <xacro:ur5_robot prefix="test" joint_limited="true"
+    <xacro:include filename="$(find mir_ur5_description)/urdf/ur5.urdf.xacro"/>
+    <xacro:ur5_robot prefix="${prefix}" joint_limited="true"
     shoulder_pan_lower_limit="${-pi}" shoulder_pan_upper_limit="${pi}"
     shoulder_lift_lower_limit="${-pi}" shoulder_lift_upper_limit="${pi}"
@@ -165,6 +165,6 @@
     <!--This joint needs to be in the mir_200_v1.urdf.xacro! Otherwise the robot cant be placed exactly on the base platform-->
     <joint name="robot_to_ur5" type="fixed">
-      <parent link="${prefix}base_footprint"/>
-      <child link="testbase_link"/>
+      <parent link="${prefix}base_link"/>
+      <child link="${prefix}base_link_ur5"/>
       <origin xyz="0.244311 -0.140242 0.450477"/>
     </joint>

Commit message: ekf is responsible for publishing the odom_comb topic. But no idea how to get that going...

File: mir_ur5_description/urdf/mir_200_v1.urdf.xacro (robot description, xacro)
@@ -154,5 +154,5 @@
     </gazebo>
     <!--Include the UR5 into the model. The position of the model was measured usind laser scanner. See Florians master thesis-->
-    <xacro:include filename="$(find mir_ur5_description)/urdf/ur5.urdf.xacro"/>
+    <!-- <xacro:include filename="$(find mir_ur5_description)/urdf/ur5.urdf.xacro"/>
     <xacro:ur5_robot prefix="${prefix}" joint_limited="true"
     shoulder_pan_lower_limit="${-pi}" shoulder_pan_upper_limit="${pi}"
@@ -162,11 +162,11 @@
     wrist_2_lower_limit="${-pi}" wrist_2_upper_limit="${pi}"
     wrist_3_lower_limit="${-pi}" wrist_3_upper_limit="${pi}"
-    transmission_hw_interface="$(arg transmission_hw_interface)"/>
+    transmission_hw_interface="$(arg transmission_hw_interface)"/> -->
     <!--This joint needs to be in the mir_200_v1.urdf.xacro! Otherwise the robot cant be placed exactly on the base platform-->
-    <joint name="robot_to_ur5" type="fixed">
+    <!-- <joint name="robot_to_ur5" type="fixed">
       <parent link="${prefix}base_link"/>
       <child link="${prefix}base_link_ur5"/>
       <origin xyz="0.244311 -0.140242 0.450477"/>
-    </joint>
+    </joint> -->
     <!-- IMU -->
     <joint name="${prefix}base_link_to_imu_joint" type="fixed">

Commit message: Cleaned mir_ur5.launch and started implementing the arm Set gazebo start to paused Tried using the pid params. But dont use!!! Copied some files in this repo Changed some params in the mir_200.transmision.xacro Removed the ur from the mir_200_v1 and put it in the mir_ur5.xacro where it belongs

File: mir_ur5_description/urdf/mir_200_v1.urdf.xacro (robot description, xacro)
@@ -4,9 +4,9 @@
   xmlns:sensor="http://playerstage.sourceforge.net/gazebo/xmlschema/#sensor"
   xmlns:xacro="http://ros.org/wiki/xacro">
-  <xacro:include filename="$(find mir_description)/urdf/include/common_properties.urdf.xacro" />
-  <xacro:include filename="$(find mir_description)/urdf/include/imu.gazebo.urdf.xacro" />
-  <xacro:include filename="$(find mir_description)/urdf/include/mir_200.gazebo.xacro" />
-  <xacro:include filename="$(find mir_description)/urdf/include/mir_200.transmission.xacro" />
-  <xacro:include filename="$(find mir_description)/urdf/include/sick_s300.urdf.xacro" />
+  <xacro:include filename="$(find mir_ur5_description)/urdf/include/common_properties.urdf.xacro" />
+  <xacro:include filename="$(find mir_ur5_description)/urdf/include/imu.gazebo.urdf.xacro" />
+  <xacro:include filename="$(find mir_ur5_description)/urdf/include/mir_200.gazebo.xacro" />
+  <xacro:include filename="$(find mir_ur5_description)/urdf/include/mir_200.transmission.xacro" />
+  <xacro:include filename="$(find mir_ur5_description)/urdf/include/sick_s300.urdf.xacro" />
   <xacro:property name="deg_to_rad" value="0.017453293" />
   <xacro:property name="mir_200_base_mass" value="58.0" />
@@ -153,20 +153,4 @@
       <material>Gazebo/LightGrey</material>
     </gazebo>
-    <!--Include the UR5 into the model. The position of the model was measured usind laser scanner. See Florians master thesis-->
-    <!-- <xacro:include filename="$(find mir_ur5_description)/urdf/ur5.urdf.xacro"/>
-    <xacro:ur5_robot prefix="${prefix}" joint_limited="true"
-    shoulder_pan_lower_limit="${-pi}" shoulder_pan_upper_limit="${pi}"
-    shoulder_lift_lower_limit="${-pi}" shoulder_lift_upper_limit="${pi}"
-    elbow_joint_lower_limit="${-pi}" elbow_joint_upper_limit="${pi}"
-    wrist_1_lower_limit="${-pi}" wrist_1_upper_limit="${pi}"
-    wrist_2_lower_limit="${-pi}" wrist_2_upper_limit="${pi}"
-    wrist_3_lower_limit="${-pi}" wrist_3_upper_limit="${pi}"
-    transmission_hw_interface="$(arg transmission_hw_interface)"/> -->
-    <!--This joint needs to be in the mir_200_v1.urdf.xacro! Otherwise the robot cant be placed exactly on the base platform-->
-    <!-- <joint name="robot_to_ur5" type="fixed">
-      <parent link="${prefix}base_link"/>
-      <child link="${prefix}base_link_ur5"/>
-      <origin xyz="0.244311 -0.140242 0.450477"/>
-    </joint> -->
     <!-- IMU -->
     <joint name="${prefix}base_link_to_imu_joint" type="fixed">

File: mir_ur5_description/urdf/mir_ur5.urdf.xacro (robot description, xacro)
@@ -2,5 +2,5 @@
 <robot xmlns:controller="http://playerstage.sourceforge.net/gazebo/xmlschema/#controller"
         xmlns:interface="http://playerstage.sourceforge.net/gazebo/xmlschema/#interface"
-        xmlns:xacro="http://ros.org/wiki/xacro"
+        xmlns:xacro="http://wiki.ros.org/xacro"
         xmlns:sensor="http://playerstage.sourceforge.net/gazebo/xmlschema/#sensor"
         name="MiR200_UR5">
@@ -10,16 +10,26 @@
     <!-- <xacro:property name="robot_name" value='$(arg robot_name)'/> -->
     <!--Include all needed urdf files-->
-    <!--Include urdf of the MiR base-->
     <xacro:include filename="$(find mir_ur5_description)/urdf/mir_200_v1.urdf.xacro"/>
+    <xacro:include filename="$(find mir_ur5_description)/urdf/ur5.urdf.xacro"/>
     <xacro:mir_200 prefix=""/>
+    <!-- <xacro:ur5_robot prefix="" joint_limited="true"/> -->
+    <!--The position of the model was measured usind laser scanner. See Florians master thesis-->
+    <!-- <joint name="robot_to_ur5" type="fixed">
+      <parent link="base_link"/>
+      <child link="base_link_ur5"/>
+      <origin xyz="0.244311 -0.140242 0.450477" rpy="0.0 0.0 0.0"/>
+    </joint> -->
     <!--Link to Gazebo library-->
     <gazebo>
         <plugin name="gazebo_ros_control" filename="libgazebo_ros_control.so">
-            <!-- <xacro:unless value="${robot_namespace == ''}">
-                <robotNamespace>$(arg robot_namespace)</robotNamespace>
-            </xacro:unless> -->
             <controlPeriod>0.001</controlPeriod>
             <legacyModeNS>true</legacyModeNS>
         </plugin>
     </gazebo>
+    <!-- Either use the part in the <gazebo> tags or the following -->
+    <!-- <xacro:diff_controller_plugin_gazebo prefix=""
+        left_wheel_joint="left_wheel_joint"
+        right_wheel_joint="right_wheel_joint"
+        wheel_separation="${2*mir_200_act_wheel_dy}"
+        wheel_radius="${mir_200_act_wheel_radius}"/> -->
 </robot>

Commit message: Added LQ file to the meshes folder Necessary because took some nodes too long for the HQ meshes

File: mir_ur5_description/urdf/mir_200_v1.urdf.xacro (robot description, xacro)
@@ -139,5 +139,5 @@
         <origin xyz="${mir_200_act_wheel_dx} 0 0" rpy="${pi/2} 0 ${pi/2}" />
         <geometry>
-          <mesh filename="package://mir_ur5_description/meshes/MiR200_UR5_base.stl" scale="0.001 0.001 0.001"/> <!--Scale is necessary because stl was generated in mm (correct dimensions) but stl has no measurements and mm are interpreted as m in gazebo-->
+          <mesh filename="package://mir_ur5_description/meshes/MiR200_UR5_base_LQ.stl" scale="0.001 0.001 0.001"/> <!--Scale is necessary because stl was generated in mm (correct dimensions) but stl has no measurements and mm are interpreted as m in gazebo-->
         </geometry>
         <xacro:insert_block name="material_white" />
@@ -146,5 +146,5 @@
         <origin xyz="${mir_200_act_wheel_dx} 0 0" rpy="${pi/2} 0 ${pi/2}" />
         <geometry>
-          <mesh filename="package://mir_ur5_description/meshes/MiR200_UR5_base.stl" scale="0.001 0.001 0.001"/> <!--Scale is necessary because stl was generated in mm (correct dimensions) but stl has no measurements and mm are interpreted as m in gazebo-->
+          <mesh filename="package://mir_ur5_description/meshes/MiR200_UR5_base_LQ.stl" scale="0.001 0.001 0.001"/> <!--Scale is necessary because stl was generated in mm (correct dimensions) but stl has no measurements and mm are interpreted as m in gazebo-->
         </geometry>
       </collision>

Commit message: Inserted tf_prefix into urdf Removed tf_prefix from robot_state_publisher Added tf_prefix in multiple places Not working, map frame is missing. No idea why

File: mir_ur5_description/urdf/mir_200_v1.urdf.xacro (robot description, xacro)
@@ -219,5 +219,5 @@
     <p3d_base_controller prefix="${prefix}" />
     <!-- Camera -->
-    <link name="camera_link">
+    <link name="${prefix}camera_link">
       <collision>
         <origin xyz="0 0 0" rpy="0 0 0"/>
@@ -238,20 +238,20 @@
       </inertial>
     </link>
-    <joint name="camera_joint" type="fixed">
+    <joint name="${prefix}camera_joint" type="fixed">
       <axis xyz="0 1 0" />
       <origin xyz="0.42 0 0.27" rpy="0 0.2 0"/> <!--set the position of the realsense-->
       <parent link="${prefix}base_link"/>
-      <child link="camera_link"/>
+      <child link="${prefix}camera_link"/>
     </joint>
     <!-- generate an optical frame http://www.ros.org/reps/rep-0103.html#suffix-frames
         so that ros and opencv can operate on the camera frame correctly -->
-    <joint name="camera_optical_joint" type="fixed">
+    <joint name="${prefix}camera_optical_joint" type="fixed">
       <!-- these values have to be these values otherwise the gazebo camera image
           won't be aligned properly with the frame it is supposedly originating from -->
       <origin xyz="0 0 0" rpy="-1.5708 0 -1.5708"/>
-      <parent link="camera_link"/>
-      <child link="camera_link_optical"/>
-    </joint>
-    <link name="camera_link_optical">
+      <parent link="${prefix}camera_link"/>
+      <child link="${prefix}camera_link_optical"/>
+    </joint>
+    <link name="${prefix}camera_link_optical">
     </link>
   </xacro:macro>

File: mir_ur5_description/urdf/mir_ur5.urdf.xacro (robot description, xacro)
@@ -13,9 +13,9 @@
     <!-- <xacro:include filename="$(find mir_ur5_description)/urdf/ur5.urdf.xacro"/> -->
     <xacro:include filename="$(find mir_ur5_description)/urdf/ur5_robot.urdf.xacro"/>
-    <xacro:mir_200 prefix=""/>
+    <xacro:mir_200 prefix="$(arg tf_prefix)"/>
     <!--The position of the model was measured usind laser scanner. See Florians master thesis-->
     <joint name="robot_to_ur5" type="fixed">
-      <parent link="base_link"/>
-      <child link="base_link_ur5"/>
+      <parent link="$(arg tf_prefix)base_link"/>
+      <child link="$(arg tf_prefix)base_link_ur5"/>
       <origin xyz="0.244311 -0.140242 0.450477" rpy="0.0 0.0 0.0"/>
     </joint>

File: mir_ur5_description/urdf/ur5_robot.urdf.xacro (robot description, xacro)
@@ -9,5 +9,5 @@
   <xacro:include filename="$(find mir_ur5_description)/urdf/ur5.urdf.xacro" />
   <!-- arm -->
-  <xacro:ur5_robot prefix="" joint_limited="false" transmission_hw_interface="$(arg transmission_hw_interface)"/>
+  <xacro:ur5_robot prefix="$(arg tf_prefix)" joint_limited="false" transmission_hw_interface="$(arg transmission_hw_interface)"/>
   <!-- <link name="world" />
   <joint name="world_joint" type="fixed">
