Commit message: First working project

File: mir_ur5_description/urdf/mir_ur5.urdf.xacro (robot description, xacro)
@@ -1,8 +1,22 @@
 <?xml version="1.0"?>
 <robot name="MiR200_UR5" xmlns:xacro="http://www.ros.org/wiki/xacro">
+    <arg name="robot_namespace" default=''/>
+    <arg name="test" default='0.002'/>
+    <xacro:property name="robot_namespace" value='$(arg robot_namespace)'/>
+    <xacro:property name="test" value='$(arg test)'/>
     <!--Include all needed urdf files-->
     <!--Include urdf of the MiR base-->
-    <xacro:include filename="$(find mir_description)/urdf/mir.urdf.xacro"/>
+    <xacro:include filename="$(find mir_description)/urdf/include/mir_200_v1.urdf.xacro"/>
+    <xacro:mir_200 prefix=""/>
     <!--Include urdf of the UR5 robot arm-->
-    <xacro:mir_200/> <!--Make namespace and name variable in future-->
+    <!--Link to Gazebo library-->
+    <gazebo>
+        <plugin name="gazebo_ros_control" filename="libgazebo_ros_control.so">
+            <xacro:unless value="${robot_namespace == ''}">
+                <robotNamespace>$(arg robot_namespace)</robotNamespace>
+            </xacro:unless>
+            <controlPeriod>$(arg test)</controlPeriod>
+            <legacyModeNS>true</legacyModeNS>
+        </plugin>
+    </gazebo>
 </robot>

Commit message: Added joints But Joint_state_publisher is crashing

File: mir_ur5_description/urdf/mir_ur5.urdf.xacro (robot description, xacro)
@@ -1,20 +1,28 @@
 <?xml version="1.0"?>
 <robot name="MiR200_UR5" xmlns:xacro="http://www.ros.org/wiki/xacro">
-    <arg name="robot_namespace" default=''/>
-    <arg name="test" default='0.002'/>
-    <xacro:property name="robot_namespace" value='$(arg robot_namespace)'/>
-    <xacro:property name="test" value='$(arg test)'/>
+    <arg name="robot_name" default=''/>
+    <xacro:arg name="transmission_hw_interface" default="hardware_interface/PositionJointInterface"/>
+    <xacro:property name="robot_name" value='$(arg robot_name)'/>
     <!--Include all needed urdf files-->
     <!--Include urdf of the MiR base-->
     <xacro:include filename="$(find mir_description)/urdf/include/mir_200_v1.urdf.xacro"/>
-    <xacro:mir_200 prefix=""/>
+    <xacro:mir_200 prefix="$(arg robot_name)"/>
     <!--Include urdf of the UR5 robot arm-->
+    <!--xacro:include filename="$(find ur_description)/urdf/ur5.urdf.xacro"/-->
+    <!--xacro:ur5_robot prefix="" joint_limited="true"
+    shoulder_pan_lower_limit="${-pi}" shoulder_pan_upper_limit="${pi}"
+    shoulder_lift_lower_limit="${-pi}" shoulder_lift_upper_limit="${pi}"
+    elbow_joint_lower_limit="${-pi}" elbow_joint_upper_limit="${pi}"
+    wrist_1_lower_limit="${-pi}" wrist_1_upper_limit="${pi}"
+    wrist_2_lower_limit="${-pi}" wrist_2_upper_limit="${pi}"
+    wrist_3_lower_limit="${-pi}" wrist_3_upper_limit="${pi}"
+    transmission_hw_interface="$(arg transmission_hw_interface)"/-->
     <!--Link to Gazebo library-->
     <gazebo>
         <plugin name="gazebo_ros_control" filename="libgazebo_ros_control.so">
-            <xacro:unless value="${robot_namespace == ''}">
-                <robotNamespace>$(arg robot_namespace)</robotNamespace>
+            <xacro:unless value="${robot_name == ''}">
+                <robotNamespace>$(arg robot_name)</robotNamespace>
             </xacro:unless>
-            <controlPeriod>$(arg test)</controlPeriod>
+            <controlPeriod>0.001</controlPeriod>
             <legacyModeNS>true</legacyModeNS>
         </plugin>

Commit message: Robot arm is on the plattform but in the wrong file currently only hardcoded onto the base_link

File: mir_ur5_description/urdf/mir_ur5.urdf.xacro (robot description, xacro)
@@ -9,6 +9,6 @@
     <xacro:mir_200 prefix="$(arg robot_name)"/>
     <!--Include urdf of the UR5 robot arm-->
-    <!--xacro:include filename="$(find ur_description)/urdf/ur5.urdf.xacro"/-->
-    <!--xacro:ur5_robot prefix="" joint_limited="true"
+    <xacro:include filename="$(find ur_description)/urdf/ur5.urdf.xacro"/>
+    <xacro:ur5_robot prefix="" joint_limited="true"
     shoulder_pan_lower_limit="${-pi}" shoulder_pan_upper_limit="${pi}"
     shoulder_lift_lower_limit="${-pi}" shoulder_lift_upper_limit="${pi}"
@@ -17,5 +17,11 @@
     wrist_2_lower_limit="${-pi}" wrist_2_upper_limit="${pi}"
     wrist_3_lower_limit="${-pi}" wrist_3_upper_limit="${pi}"
-    transmission_hw_interface="$(arg transmission_hw_interface)"/-->
+    transmission_hw_interface="$(arg transmission_hw_interface)"/>
+    <!--This joint needs to be in the mir_200_v1.urdf.xacro! Otherwise the robot cant be placed exactly on the base platform-->
+    <joint name="robot_to_ur5" type="fixed">
+        <parent link="base_link"/>
+        <child link="robot1base_footprint"/>
+        <origin xyz="0 0 -0.36"/>
+    </joint>
     <!--Link to Gazebo library-->
     <gazebo>

Commit message: put robot in urdf

File: mir_ur5_description/urdf/mir_ur5.urdf.xacro (robot description, xacro)
@@ -6,8 +6,9 @@
     <!--Include all needed urdf files-->
     <!--Include urdf of the MiR base-->
-    <xacro:include filename="$(find mir_description)/urdf/include/mir_200_v1.urdf.xacro"/>
+    <!--xacro:include filename="$(find mir_description)/urdf/include/mir_200_v1.urdf.xacro"/-->
+    <xacro:include filename="$(find mir_ur5_description)/urdf/mir_200_v1.urdf.xacro"/>
     <xacro:mir_200 prefix="$(arg robot_name)"/>
     <!--Include urdf of the UR5 robot arm-->
-    <xacro:include filename="$(find ur_description)/urdf/ur5.urdf.xacro"/>
+    <!--xacro:include filename="$(find ur_description)/urdf/ur5.urdf.xacro"/>
     <xacro:ur5_robot prefix="" joint_limited="true"
     shoulder_pan_lower_limit="${-pi}" shoulder_pan_upper_limit="${pi}"
@@ -17,11 +18,11 @@
     wrist_2_lower_limit="${-pi}" wrist_2_upper_limit="${pi}"
     wrist_3_lower_limit="${-pi}" wrist_3_upper_limit="${pi}"
-    transmission_hw_interface="$(arg transmission_hw_interface)"/>
+    transmission_hw_interface="$(arg transmission_hw_interface)"/-->
     <!--This joint needs to be in the mir_200_v1.urdf.xacro! Otherwise the robot cant be placed exactly on the base platform-->
-    <joint name="robot_to_ur5" type="fixed">
+    <!--joint name="robot_to_ur5" type="fixed">
         <parent link="base_link"/>
         <child link="robot1base_footprint"/>
         <origin xyz="0 0 -0.36"/>
-    </joint>
+    </joint-->
     <!--Link to Gazebo library-->
     <gazebo>

Commit message: Differed name, namespace and tf prefix

File: mir_ur5_description/urdf/mir_ur5.urdf.xacro (robot description, xacro)
@@ -1,10 +1,11 @@
 <?xml version="1.0"?>
-<robot name="MiR200_UR5" xmlns:xacro="http://www.ros.org/wiki/xacro">
+<robot name="MiR200_UR5" xmlns:xacro="http://ros.org/wiki/xacro">
     <arg name="robot_name" default=''/>
+    <arg name="robot_namespace" default=''/>
     <xacro:arg name="transmission_hw_interface" default="hardware_interface/PositionJointInterface"/>
     <xacro:property name="robot_name" value='$(arg robot_name)'/>
+    <xacro:property name="robot_namespace" value="$(arg robot_namespace)"/>
     <!--Include all needed urdf files-->
     <!--Include urdf of the MiR base-->
-    <!--xacro:include filename="$(find mir_description)/urdf/include/mir_200_v1.urdf.xacro"/-->
     <xacro:include filename="$(find mir_ur5_description)/urdf/mir_200_v1.urdf.xacro"/>
     <xacro:mir_200 prefix="$(arg robot_name)"/>
@@ -28,6 +29,6 @@
     <gazebo>
         <plugin name="gazebo_ros_control" filename="libgazebo_ros_control.so">
-            <xacro:unless value="${robot_name == ''}">
-                <robotNamespace>$(arg robot_name)</robotNamespace>
+            <xacro:unless value="${robot_namespace == ''}">
+                <robotNamespace>$(arg robot_namespace)</robotNamespace>
             </xacro:unless>
             <controlPeriod>0.001</controlPeriod>

Commit message: Copied all files that are called for the basics into own repo

File: mir_ur5_description/urdf/mir_ur5.urdf.xacro (robot description, xacro)
@@ -1,36 +1,22 @@
 <?xml version="1.0"?>
-<robot name="MiR200_UR5" xmlns:xacro="http://ros.org/wiki/xacro">
+<robot xmlns:controller="http://playerstage.sourceforge.net/gazebo/xmlschema/#controller"
+        xmlns:interface="http://playerstage.sourceforge.net/gazebo/xmlschema/#interface"
+        xmlns:xacro="http://ros.org/wiki/xacro"
+        xmlns:sensor="http://playerstage.sourceforge.net/gazebo/xmlschema/#sensor"
+        name="MiR200_UR5">
     <xacro:arg name="robot_name" default=''/>
-    <xacro:arg name="robot_namespace" default=''/>
     <xacro:arg name="tf_prefix" default=''/>
     <xacro:arg name="transmission_hw_interface" default="hardware_interface/PositionJointInterface"/>
-    <xacro:property name="robot_name" value='$(arg robot_name)'/>
-    <xacro:property name="robot_namespace" value="$(arg robot_namespace)"/>
+    <!-- <xacro:property name="robot_name" value='$(arg robot_name)'/> -->
     <!--Include all needed urdf files-->
     <!--Include urdf of the MiR base-->
     <xacro:include filename="$(find mir_ur5_description)/urdf/mir_200_v1.urdf.xacro"/>
     <xacro:mir_200 prefix=""/>
-    <!--Include urdf of the UR5 robot arm-->
-    <!--xacro:include filename="$(find ur_description)/urdf/ur5.urdf.xacro"/>
-    <xacro:ur5_robot prefix="" joint_limited="true"
-    shoulder_pan_lower_limit="${-pi}" shoulder_pan_upper_limit="${pi}"
-    shoulder_lift_lower_limit="${-pi}" shoulder_lift_upper_limit="${pi}"
-    elbow_joint_lower_limit="${-pi}" elbow_joint_upper_limit="${pi}"
-    wrist_1_lower_limit="${-pi}" wrist_1_upper_limit="${pi}"
-    wrist_2_lower_limit="${-pi}" wrist_2_upper_limit="${pi}"
-    wrist_3_lower_limit="${-pi}" wrist_3_upper_limit="${pi}"
-    transmission_hw_interface="$(arg transmission_hw_interface)"/-->
-    <!--This joint needs to be in the mir_200_v1.urdf.xacro! Otherwise the robot cant be placed exactly on the base platform-->
-    <!--joint name="robot_to_ur5" type="fixed">
-        <parent link="base_link"/>
-        <child link="robot1base_footprint"/>
-        <origin xyz="0 0 -0.36"/>
-    </joint-->
     <!--Link to Gazebo library-->
     <gazebo>
         <plugin name="gazebo_ros_control" filename="libgazebo_ros_control.so">
-            <xacro:unless value="${robot_namespace == ''}">
+            <!-- <xacro:unless value="${robot_namespace == ''}">
                 <robotNamespace>$(arg robot_namespace)</robotNamespace>
-            </xacro:unless>
+            </xacro:unless> -->
             <controlPeriod>0.001</controlPeriod>
             <legacyModeNS>true</legacyModeNS>

Commit message: Removed unnecessary comments Removed the second mir plattform again Tried the original launch ffrom the ur launch but didnt work Added robot arm again

File: mir_ur5_description/urdf/mir_ur5.urdf.xacro (robot description, xacro)
@@ -13,14 +13,15 @@
     <xacro:include filename="$(find mir_ur5_description)/urdf/ur5.urdf.xacro"/>
     <xacro:mir_200 prefix=""/>
-    <!-- <xacro:ur5_robot prefix="" joint_limited="true"/> -->
+    <xacro:ur5_robot prefix="" joint_limited="true"/>
     <!--The position of the model was measured usind laser scanner. See Florians master thesis-->
-    <!-- <joint name="robot_to_ur5" type="fixed">
+    <joint name="robot_to_ur5" type="fixed">
       <parent link="base_link"/>
       <child link="base_link_ur5"/>
       <origin xyz="0.244311 -0.140242 0.450477" rpy="0.0 0.0 0.0"/>
-    </joint> -->
+    </joint>
     <!--Link to Gazebo library-->
     <gazebo>
         <plugin name="gazebo_ros_control" filename="libgazebo_ros_control.so">
+            <!-- <robotSimType>gazebo_ros_control/DefaultRobotHWSim</robotSimType> -->
             <controlPeriod>0.001</controlPeriod>
             <legacyModeNS>true</legacyModeNS>

Commit message: Handed over tf_prefix to ur5 explicitly. Commente some unecessary links and joints

File: mir_ur5_description/urdf/mir_ur5.urdf.xacro (robot description, xacro)
@@ -12,5 +12,7 @@
     <xacro:include filename="$(find mir_ur5_description)/urdf/mir_200_v1.urdf.xacro"/>
     <!-- <xacro:include filename="$(find mir_ur5_description)/urdf/ur5.urdf.xacro"/> -->
-    <xacro:include filename="$(find mir_ur5_description)/urdf/ur5_robot.urdf.xacro"/>
+    <xacro:include filename="$(find mir_ur5_description)/urdf/ur5_robot.urdf.xacro">
+        <arg name="tf_prefix" value="$(arg tf_prefix)"/>
+    </xacro:include>
     <xacro:mir_200 prefix="$(arg tf_prefix)"/>
     <!--The position of the model was measured usind laser scanner. See Florians master thesis-->

File: mir_ur5_description/urdf/ur5.urdf.xacro (robot description, xacro)
@@ -295,21 +295,17 @@
     <xacro:ur_arm_gazebo prefix="${prefix}" />
     <!-- ROS base_link to UR 'Base' Coordinates transform -->
-    <link name="${prefix}base_ur5"/>
-    <joint name="${prefix}base_link_ur5-base_fixed_joint" type="fixed">
-      <!-- NOTE: this rotation is only needed as long as base_link_ur5 itself is
-                 not corrected wrt the real robot (ie: rotated over 180
-                 degrees)
-      -->
+    <!-- <link name="${prefix}base_ur5"/> -->
+    <!-- <joint name="${prefix}base_link_ur5-base_fixed_joint" type="fixed">
       <origin xyz="0 0 0" rpy="0 0 ${-pi}"/>
       <parent link="${prefix}base_link_ur5"/>
       <child link="${prefix}base_ur5"/>
-    </joint>
+    </joint> -->
     <!-- Frame coincident with all-zeros TCP on UR controller -->
-    <link name="${prefix}tool0"/>
+    <!-- <link name="${prefix}tool0"/>
     <joint name="${prefix}wrist_3_link_ur5-tool0_fixed_joint" type="fixed">
       <origin xyz="0 ${wrist_3_length} 0" rpy="${pi/-2.0} 0 0"/>
       <parent link="${prefix}wrist_3_link_ur5"/>
       <child link="${prefix}tool0"/>
-    </joint>
+    </joint> -->
   </xacro:macro>
 </robot>

File: mir_ur5_description/urdf/ur5_robot.urdf.xacro (robot description, xacro)
@@ -4,4 +4,5 @@
        name="ur5" >
   <xacro:arg name="transmission_hw_interface" default="hardware_interface/PositionJointInterface"/>
+  <xacro:arg name="tf_prefix" default=""/>
   <!-- common stuff -->
   <!-- <xacro:include filename="$(find ur_description)/urdf/common.gazebo.xacro" /> -->
