Commit message: Removed unnecessary / Rolled back to maze world for laser scanner data Removed / in /map in amcl Removed unnecessary / in start_maps

File: mir_ur5_description/urdf/include/imu.gazebo.urdf.xacro (robot description, xacro)
@@ -8,5 +8,5 @@
   </xacro:if>
   <xacro:unless value="${tf_prefix == ''}">
-      <xacro:property name="imu_frame" value="$(arg tf_prefix)/imu_frame" />
+      <xacro:property name="imu_frame" value="$(arg tf_prefix)imu_frame" />
   </xacro:unless>
   <xacro:macro name="imu_gazebo" params="link imu_topic update_rate stdev">
