Commit message: Finished deleting all hard-coded tf prefixes and use args Removed obsolete code Created lauch for moveit stuff Changed the srdf for moveit to be a srdf.xacro so it takes args
Still need to refactor everything

File: mir_ur5_description/urdf/include/sick_s300.urdf.xacro (robot description, xacro)
@@ -6,6 +6,6 @@
   <xacro:property name="laser_z" value="0.185" />
   <xacro:property name="laser_mass" value="2.0" />
-  <xacro:macro name="sick_s300" params="link topic prefix">
-    <link name="${prefix}${link}">
+  <xacro:macro name="sick_s300" params="link topic tf_prefix">
+    <link name="${tf_prefix}${link}">
       <visual>
         <origin xyz="0.0 0.0 0.0" rpy="${pi} 0 0" />
@@ -26,8 +26,8 @@
       </xacro:box_inertial>
     </link>
-    <gazebo reference="${prefix}${link}">
+    <gazebo reference="${tf_prefix}${link}">
       <!-- <material value="Gazebo/Yellow" /> -->
       <material value="Gazebo/FlatBlack" />
-      <sensor type="gpu_ray" name="${prefix}${link}">
+      <sensor type="gpu_ray" name="${tf_prefix}${link}">
         <pose>0 0 0 0 0 0</pose>
         <visualize>false</visualize>
@@ -57,6 +57,6 @@
         </ray>
         <plugin name="gazebo_ros_${link}_controller" filename="libgazebo_ros_gpu_laser.so">
-          <!-- no prefix, plugin always uses a tf_prefix (if none is set it uses robotNamespace) -->
-          <frameName>/robot1_tf/${link}</frameName>
+          <!-- no tf_prefix, plugin always uses a tf_prefix (if none is set it uses robotNamespace) -->
+          <frameName>/${tf_prefix}${link}</frameName>
           <topicName>${topic}</topicName>
         </plugin>

File: mir_ur5_description/urdf/mir_200_v1.urdf.xacro (robot description, xacro)
@@ -180,5 +180,5 @@
       <origin xyz="0.4288 0.2358 0.1914" rpy="0.0 0.0 ${0.25 * pi}" />  <!-- from visually matching up the meshes of the MiR and the laser scanner -->
     </joint>
-    <xacro:sick_s300 prefix="${prefix}" link="front_laser_link" topic="f_scan" />
+    <xacro:sick_s300 tf_prefix="${prefix}" link="front_laser_link" topic="f_scan" />
     <joint name="${prefix}base_link_to_back_laser_joint" type="fixed">
       <parent link="${prefix}base_link" />
@@ -186,5 +186,5 @@
       <origin xyz="-0.3548 -0.2352 0.1914" rpy="0.0 0.0 ${-0.75 * pi}" />  <!-- from visually matching up the meshes of the MiR and the laser scanner -->
     </joint>
-    <xacro:sick_s300 prefix="${prefix}" link="back_laser_link" topic="b_scan" />
+    <xacro:sick_s300 tf_prefix="${prefix}" link="back_laser_link" topic="b_scan" />
     <!-- Ultrasound sensors -->
     <joint name="${prefix}us_1_joint" type="fixed">   <!-- right ultrasound -->
