Commit message: Give the blocks to pick up a mu to increase friction Maybe separated block will no longer drift apart

File: control_ur5_test/urdf/separated_block.urdf.xacro (robot description, xacro)
@@ -21,7 +21,11 @@
         </inertial>
     </link>
-    <!-- <gazebo reference="box_base">
-        <kp>0.0</kp>
-    </gazebo> -->
+    <gazebo reference="box_base">
+        <material>Gazebo/DarkGrey</material>
+        <mu1 value="100000.0"/>
+        <mu2 value="100000.0"/>
+        <kp value="10000000.0"/>
+        <kd value="1.0"/>
+    </gazebo>
     <link name="box_base_movable">
         <visual>
@@ -41,7 +45,11 @@
         </inertial>
     </link>
-    <!-- <gazebo reference="box_base_movable">
-        <kp>0.0</kp>
-    </gazebo> -->
+    <gazebo reference="box_base_movable">
+        <material>Gazebo/DarkGrey</material>
+        <mu1 value="100000.0"/>
+        <mu2 value="100000.0"/>
+        <kp value="10000000.0"/>
+        <kd value="1.0"/>
+    </gazebo>
     <joint name="block_joint" type="prismatic">
         <parent link="box_base" />
