Commit message: Played with the gazebo parameters for the models Put maxVel= 0 in. I think this was the solution Changed the size of the object Inserted Parameters for the joint in the separated block

File: control_ur5_test/urdf/block.urdf (robot description, URDF)
Before this commit: robot box, 1 links, 0 joints
Links:
- link box_base: geometry collision box size=3.0 1.0 0.1; visual box size=3.0 1.0 0.1

File: control_ur5_test/urdf/separated_block.urdf.xacro (robot description, xacro)
@@ -1,6 +1,6 @@
 <?xml version="1.0"?>
 <robot name="box" xmlns:xacro="http://wiki.ros.org/xacro">
-    <xacro:property name="x_size" value="0.5"/>
-    <xacro:property name="y_size" value="0.5"/>
+    <xacro:property name="x_size" value="3.0"/>
+    <xacro:property name="y_size" value="1.0"/>
     <xacro:property name="z_size" value="0.1"/>
     <link name="box_base">
@@ -23,8 +23,10 @@
     <gazebo reference="box_base">
         <material>Gazebo/DarkGrey</material>
-        <mu1 value="100000.0"/>
-        <mu2 value="100000.0"/>
-        <kp value="10000000.0"/>
-        <kd value="1.0"/>
+        <mu1 value="10000000000.0"/>
+        <mu2 value="10000000000.0"/>
+        <kp value="10000.0"/>
+        <kd value="1000.0"/>
+        <maxVel value="0"/>
+        <!-- <minDepth value="0.1"/> -->
     </gazebo>
     <link name="box_base_movable">
@@ -47,8 +49,10 @@
     <gazebo reference="box_base_movable">
         <material>Gazebo/DarkGrey</material>
-        <mu1 value="100000.0"/>
-        <mu2 value="100000.0"/>
-        <kp value="10000000.0"/>
-        <kd value="1.0"/>
+        <mu1 value="10000000000.0"/>
+        <mu2 value="10000000000.0"/>
+        <kp value="10000.0"/>
+        <kd value="1000.0"/>
+        <maxVel value="0"/>
+        <!-- <minDepth value="0.1"/> -->
     </gazebo>
     <joint name="block_joint" type="prismatic">
@@ -60,3 +64,16 @@
         <dynamics damping="0.01" friction="0.5"/>
     </joint>
+    <gazebo reference="block_joint">
+        <stopCfm value="0.8"/>
+        <stopErp value="0"/>
+        <provideFeedback value="true"/>
+        <implicitSpringDamper value="true"/>
+    </gazebo>
+    <gazebo>
+        <plugin name="ft_sensor" filename="libgazebo_ros_ft_sensor.so">
+            <updateRate>100.0</updateRate>
+            <topicName>ft_sensor_topic</topicName>
+            <jointName>block_joint</jointName>
+        </plugin>
+    </gazebo>
 </robot>
